File: Option1/Option1.kicad_pcb (KiCad board)
At the start: 2 copper layers, 0 parts

Commit message: USB Schaltung angepasst, Transistoren korrigiert, Stecker ausgetauscht, Dioden hinzugefügt
Other:
- board outline added: 86 x 62 mm
Changed lines of the file:
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@@
 	)
 	(net 0 "")
+	(gr_rect
+		(start 100 50)
+		(end 186 112)
+		(stroke
+			(width 0.05)
+			(type default)
+		)
+		(fill no)
+		(layer "Edge.Cuts")
+	)
 	(embedded_fonts no)
 )
