File: Option1/CAN.kicad_sch (KiCad schematic)
At the start: 10 parts, among them U301 TJA1051T-3, U302 MCP2515-I/ST, X301 XL1EL89CSI-111YLC-8M

Commit message: Schaltplan zu bachelorarbeit Dokument hinzuigefügt. Fertigf bis SPI Flash
Other:
- moved on the sheet: C301, C302
Changed lines of the file:
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@@
 	)
 	(junction
-		(at 156.21 121.92)
+		(at 162.56 121.92)
 		(diameter 0)
 		(color 0 0 0 0)
 	)
 	(junction
-		(at 191.77 78.74)
+		(at 151.13 121.92)
 		(diameter 0)
 		(color 0 0 0 0)
@@
 	)
 	(junction
+		(at 151.13 99.06)
+		(diameter 0)
+		(color 0 0 0 0)
+	)
+	(junction
+		(at 193.04 78.74)
+		(diameter 0)
+		(color 0 0 0 0)
+	)
+	(junction
 		(at 177.8 116.84)
 		(diameter 0)
@@
 	)
 	(junction
-		(at 167.64 121.92)
-		(diameter 0)
-		(color 0 0 0 0)
-	)
-	(junction
 		(at 170.18 116.84)
 		(diameter 0)
 		(color 0 0 0 0)
 	)
-	(junction
-		(at 156.21 99.06)
-		(diameter 0)
-		(color 0 0 0 0)
-	)
 	(wire
 		(pts
@@
 	(wire
 		(pts
-			(xy 191.77 99.06) (xy 191.77 78.74)
-		)
-		(stroke
-			(width 0)
-			(type default)
-		)
-	)
-	(wire
-		(pts
-			(xy 156.21 111.76) (xy 156.21 121.92)
+			(xy 151.13 111.76) (xy 151.13 121.92)
 		)
 		(stroke
@@
 	(wire
 		(pts
-			(xy 187.96 78.74) (xy 191.77 78.74)
+			(xy 187.96 78.74) (xy 193.04 78.74)
 		)
 		(stroke
@@
 	(wire
 		(pts
+			(xy 151.13 121.92) (xy 114.3 121.92)
+		)
+		(stroke
+			(width 0)
+			(type default)
+		)
+	)
+	(wire
+		(pts
 			(xy 82.55 101.6) (xy 82.55 99.06)
 		)
@@
 	(wire
 		(pts
-			(xy 156.21 99.06) (xy 127 99.06)
-		)
-		(stroke
-			(width 0)
-			(type default)
-		)
-	)
-	(wire
-		(pts
 			(xy 127 91.44) (xy 213.36 91.44)
 		)
@@
 	(wire
 		(pts
-			(xy 156.21 121.92) (xy 114.3 121.92)
-		)
-		(stroke
-			(width 0)
-			(type default)
-		)
-	)
-	(wire
-		(pts
-			(xy 167.64 121.92) (xy 156.21 121.92)
+			(xy 151.13 121.92) (xy 162.56 121.92)
 		)
 		(stroke
@@
 	(wire
 		(pts
-			(xy 156.21 99.06) (xy 156.21 104.14)
+			(xy 151.13 99.06) (xy 151.13 104.14)
 		)
 		(stroke
@@
 	(wire
 		(pts
-			(xy 191.77 78.74) (xy 247.65 78.74)
-		)
-		(stroke
-			(width 0)
-			(type default)
-		)
-	)
-	(wire
-		(pts
 			(xy 82.55 101.6) (xy 80.01 101.6)
 		)
@@
 	(wire
 		(pts
-			(xy 156.21 99.06) (xy 191.77 99.06)
-		)
-		(stroke
-			(width 0)
-			(type default)
-		)
-	)
-	(wire
-		(pts
 			(xy 265.43 78.74) (xy 265.43 93.98)
 		)
@@
 	(wire
 		(pts
+			(xy 193.04 99.06) (xy 193.04 78.74)
+		)
+		(stroke
+			(width 0)
+			(type default)
+		)
+	)
+	(wire
+		(pts
 			(xy 199.39 116.84) (xy 199.39 121.92)
 		)
@@
 	(wire
 		(pts
+			(xy 162.56 121.92) (xy 170.18 121.92)
+		)
+		(stroke
+			(width 0)
+			(type default)
+		)
+	)
+	(wire
+		(pts
 			(xy 243.84 99.06) (xy 247.65 99.06)
 		)
@@
 	(wire
 		(pts
+			(xy 193.04 78.74) (xy 247.65 78.74)
+		)
+		(stroke
+			(width 0)
+			(type default)
+		)
+	)
+	(wire
+		(pts
 			(xy 80.01 88.9) (xy 77.47 88.9)
 		)
@@
 	(wire
 		(pts
+			(xy 151.13 99.06) (xy 193.04 99.06)
+		)
+		(stroke
+			(width 0)
+			(type default)
+		)
+	)
+	(wire
+		(pts
 			(xy 243.84 106.68) (xy 247.65 106.68)
 		)
@@
 	(wire
 		(pts
-			(xy 167.64 78.74) (xy 167.64 104.14)
+			(xy 162.56 78.74) (xy 162.56 104.14)
 		)
 		(stroke
@@
 	(wire
 		(pts
+			(xy 151.13 99.06) (xy 127 99.06)
+		)
+		(stroke
+			(width 0)
+			(type default)
+		)
+	)
+	(wire
+		(pts
 			(xy 127 93.98) (xy 213.36 93.98)
 		)
@@
 	(wire
 		(pts
-			(xy 167.64 121.92) (xy 170.18 121.92)
-		)
-		(stroke
-			(width 0)
-			(type default)
-		)
-	)
-	(wire
-		(pts
 			(xy 243.84 96.52) (xy 247.65 96.52)
 		)
@@
 	(wire
 		(pts
-			(xy 167.64 111.76) (xy 167.64 121.92)
+			(xy 162.56 111.76) (xy 162.56 121.92)
 		)
 		(stroke
@@
 	(wire
 		(pts
-			(xy 167.64 78.74) (xy 114.3 78.74)
+			(xy 162.56 78.74) (xy 114.3 78.74)
 		)
 		(stroke
@@
 	)
 	(label "CAN_RX"
+		(at 205.74 93.98 0)
+		(effects
+			(font
+				(size 1.27 1.27)
+			)
+			(justify left bottom)
+		)
+	)
+	(label "CAN_RX"
 		(at 127 93.98 0)
+		(effects
+			(font
+				(size 1.27 1.27)
+			)
+			(justify left bottom)
+		)
+	)
+	(label "CAN_TX"
+		(at 205.74 91.44 0)
 		(effects
 			(font
@@
 	(symbol
 		(lib_id "easyeda2kicad:CL10B104KA8NNNC")
-		(at 167.64 107.95 90)
+		(at 162.56 107.95 90)
 		(mirror x)
 		(unit 1)
@@
 		(dnp no)
 		(property "Reference" "C301"
-			(at 165.1 106.68 90)
+			(at 160.02 106.68 90)
 			(effects
 				(font
@@
 		)
 		(property "Value" "100nF"
-			(at 165.1 109.22 90)
+			(at 160.02 109.22 90)
 			(effects
 				(font
@@
 		)
 		(property "Footprint" "easyeda2kicad:C0603"
+			(at 170.18 107.95 0)
+			(effects
+				(font
+					(size 1.27 1.27)
+				)
+				(hide yes)
+			)
+		)
+		(property "Datasheet" "https://lcsc.com/product-detail/Multilayer-Ceramic-Capacitors-MLCC-SMD-SMT_SAMSUNG_CL10B104KA8NNNC_100nF-104-10-25V_C1590.html"
+			(at 172.72 107.95 0)
+			(effects
+				(font
+					(size 1.27 1.27)
+				)
+				(hide yes)
+			)
+		)
+		(property "Description" ""
+			(at 162.56 107.95 0)
+			(effects
+				(font
+					(size 1.27 1.27)
+				)
+				(hide yes)
+			)
+		)
+		(property "LCSC Part" "C1590"
 			(at 175.26 107.95 0)
-			(effects
-				(font
-					(size 1.27 1.27)
-				)
-				(hide yes)
-			)
-		)
-		(property "Datasheet" "https://lcsc.com/product-detail/Multilayer-Ceramic-Capacitors-MLCC-SMD-SMT_SAMSUNG_CL10B104KA8NNNC_100nF-104-10-25V_C1590.html"
-			(at 177.8 107.95 0)
-			(effects
-				(font
-					(size 1.27 1.27)
-				)
-				(hide yes)
-			)
-		)
-		(property "Description" ""
-			(at 167.64 107.95 0)
-			(effects
-				(font
-					(size 1.27 1.27)
-				)
-				(hide yes)
-			)
-		)
-		(property "LCSC Part" "C1590"
-			(at 180.34 107.95 0)
 			(effects
 				(font
@@
 	(symbol
 		(lib_id "easyeda2kicad:CL10B104KA8NNNC")
-		(at 156.21 107.95 90)
+		(at 151.13 107.95 90)
 		(mirror x)
 		(unit 1)
@@
 		(dnp no)
 		(property "Reference" "C302"
-			(at 153.162 106.68 90)
+			(at 148.082 106.68 90)
 			(effects
 				(font
@@
 		)
 		(property "Value" "100nF"
-			(at 153.162 109.22 90)
+			(at 148.082 109.22 90)
 			(effects
 				(font
@@
 		)
 		(property "Footprint" "easyeda2kicad:C0603"
+			(at 158.75 107.95 0)
+			(effects
+				(font
+					(size 1.27 1.27)
+				)
+				(hide yes)
+			)
+		)
+		(property "Datasheet" "https://lcsc.com/product-detail/Multilayer-Ceramic-Capacitors-MLCC-SMD-SMT_SAMSUNG_CL10B104KA8NNNC_100nF-104-10-25V_C1590.html"
+			(at 161.29 107.95 0)
+			(effects
+				(font
+					(size 1.27 1.27)
+				)
+				(hide yes)
+			)
+		)
+		(property "Description" ""
+			(at 151.13 107.95 0)
+			(effects
+				(font
+					(size 1.27 1.27)
+				)
+				(hide yes)
+			)
+		)
+		(property "LCSC Part" "C1590"
 			(at 163.83 107.95 0)
 			(effects
 				(font
-					(size 1.27 1.27)
-				)
-				(hide yes)
-			)
-		)
-		(property "Datasheet" "https://lcsc.com/product-detail/Multilayer-Ceramic-Capacitors-MLCC-SMD-SMT_SAMSUNG_CL10B104KA8NNNC_100nF-104-10-25V_C1590.html"
-			(at 166.37 107.95 0)
-			(effects
-				(font
-					(size 1.27 1.27)
-				)
-				(hide yes)
-			)
-		)
-		(property "Description" ""
-			(at 156.21 107.95 0)
-			(effects
-				(font
-					(size 1.27 1.27)
-				)
-				(hide yes)
-			)
-		)
-		(property "LCSC Part" "C1590"
-			(at 168.91 107.95 0)
-			(effects
-				(font
